File: Hardware/SparkX_smol_Environmental.sch (EAGLE design)
At the start: 27 parts, among them U1 SGP40, U2 BME280, U3 VEML7700-TT

Commit message: Add production files and README
Parts:
- removed PROC_PWR_EN: JUMPER-SMT_2_NC_TRACE_SILK, SparkFun-Jumpers:JUMPER-SMT_2_NC_TRACE_SILK
- added R4: 4.7, SparkFun-Resistors:4.7OHM-0402T-1/16W-1%
- R1: device SparkFun-Resistors:4.7OHM-0603-1/10W-1% -> SparkFun-Resistors:4.7OHM-0402T-1/16W-1%
Connections:
- new net N$4: C5.1, C6.1, R4.1, U3.VDD
- net 3.3V: now also R4.2; no longer C5.1, C6.1, U3.VDD
- net GND: no longer PROC_PWR_EN.2
- net PROC_PWR_EN: no longer PROC_PWR_EN.1
Other:
- note added: "X01"
- note removed: "Disable Processor Board Regulator"
- note removed: "X02"
- moved on the sheet: C5, C6, JP1, R2, R3
